File: Schematics/PC6502-STORAGE/SDCard.kicad_sch (KiCad schematic)
At the start: 26 parts, among them J7 Conn_02x05_Odd_Even, J8 TF-15X15, U3 ATF1502AS, U4 TXB0108PW, U5 AMS1117-3.3

Commit message: Tidy up and simplify
Created schematic for FM & Speech sound board
Made Storage board just for Compact Flash (CF) storage
Routed Storage PCB
Parts:
- D10: now fitted
- U3: value ATF1502AS -> ATF1504AS; now fitted
Changed lines of the file:
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@@
 		(in_bom yes)
 		(on_board yes)
-		(dnp yes)
+		(dnp no)
 		(fields_autoplaced yes)
 		(property "Reference" "U3"
@@
 			)
 		)
-		(property "Value" "ATF1502AS"
+		(property "Value" "ATF1504AS"
 			(at 66.9133 48.26 0)
 			(effects
@@
 		(in_bom yes)
 		(on_board yes)
-		(dnp yes)
+		(dnp no)
 		(property "Reference" "D10"
 			(at 26.416 85.09 0)
