File: Schematics/PC6502-FM-SPEECH/PC6502-FM-SPEECH.kicad_sch (KiCad schematic)
At the start: 17 parts, among them J1 BUS, J5 Conn_02x05_Odd_Even, U1 ATF1502AS

Commit message: Updated following testing
New CPLD code for CPU and VIA
Fixed mistakes with CPU Board and upped to Rev 1.2 (My Rev 1.1 has mods on)
Updated README
Parts:
- U1: now fitted
Changed lines of the file:
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@@
 		(in_bom yes)
 		(on_board yes)
-		(dnp yes)
+		(dnp no)
 		(fields_autoplaced yes)
 		(property "Reference" "U1"
