File: Schematics/PC6502-AIISLOT/PC6502-AIISLOT.kicad_sch (KiCad schematic)
At the start: 20 parts, among them J1 BUS, J2 SLOT0, J3 SLOT1, J4 POWER IN, J5 Conn_02x05_Odd_Even, U1 ATF1502AS

Commit message: CPU CPLD UPDATE!!
CPU will now run at 14MHz with the updated code in the CPLD
Begun assembly of Speech/FM board
Other:
- note added: "FRONT"
- note added: "REAR"
Changed lines of the file:
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@@
 	(generator_version "9.0")
 	(paper "A4")
+	(text "REAR"
+		(exclude_from_sim no)
+		(at 127.762 28.702 0)
+		(effects
+			(font
+				(size 1.27 1.27)
+			)
+		)
+	)
+	(text "FRONT\n"
+		(exclude_from_sim no)
+		(at 57.15 100.838 0)
+		(effects
+			(font
+				(size 1.27 1.27)
+			)
+		)
+	)
 	(text "CPU_CLK is the stretched\nversion of CLK. \nUse nSLOW0 and nSLOW1 to\nslow the clock down"
 		(exclude_from_sim no)
 		(at 264.16 141.986 0)
+		(effects
+			(font
+				(size 1.27 1.27)
+			)
+		)
+	)
+	(text "FRONT\n"
+		(exclude_from_sim no)
+		(at 128.27 100.838 0)
 		(effects
 			(font
@@
 		(effects
 			(font
+				(size 1.27 1.27)
+			)
+		)
+	)
+	(text "REAR"
+		(exclude_from_sim no)
+		(at 57.15 27.432 0)
+		(effects
+			(font
