File: Schematics/PC6502_KEYBED/Dual_QDSP-2118.kicad_sch (KiCad schematic)
At the start: 2 parts

Commit message: Keyboard code and schematics
Updated the Schematics and have a mostly functioning keyboard (can't turn off caps lock yet)
Parts:
- DS1: value HDSP-2503 -> HDSP-2103
Changed lines of the file:
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@@
 			)
 		)
-		(property "Value" "HDSP-2503"
+		(property "Value" "HDSP-2103"
 			(at 161.29 64.77 0)
 			(effects
