File: Schematics/PC6502_KEYBED/PC6502_KEYBED.kicad_pcb (KiCad board)
At the start: 4 copper layers, 399 x 96.4 mm, 161 parts, among them J4 Conn_02x05_Odd_Even, J6 MTJ-88ARX1-FSM-LG, Q7 2N3904, Q8 2N3904, SW1 SW_Push, SW10 SW_Push, SW11 SW_Push, SW12 SW_Push, SW13 SW_Push, SW14 SW_Push, SW15 SW_Push, SW16 SW_Push, SW17 SW_Push, SW18 SW_Push, SW19 SW_Push, SW2 SW_Push, SW20 SW_Push, SW21 SW_Push, SW22 SW_Push, SW23 SW_Push, SW24 SW_Push, SW25 SW_Push, SW26 SW_Push, SW27 SW_Push, SW28 SW_Push, SW29 SW_Push, SW3 SW_Push, SW30 SW_Push, SW31 SW_Push, SW32 SW_Push, SW33 SW_Push, SW34 SW_Push, SW35 SW_Push, SW36 SW_Push, SW37 SW_Push, SW38 SW_Push, SW39 SW_Push, SW4 SW_Push, SW40 SW_Push, SW41 SW_Push, SW42 SW_Push, SW43 SW_Push, SW44 SW_Push, SW45 SW_Push, SW46 SW_Push, SW47 SW_Push, SW48 SW_Push, SW49 SW_Push, SW5 SW_Push, SW50 SW_Push, SW51 SW_Push, SW52 SW_Push, SW53 SW_Push, SW54 SW_Push, SW55 SW_Push, SW56 SW_Push, SW57 SW_Push, SW58 SW_Push, SW59 SW_Push, SW6 SW_Push, SW60 SW_Push, SW61 SW_Push, SW62 SW_Push, SW63 SW_Push, SW64 SW_Push, SW65 SW_Push, SW7 SW_Push, SW8 SW_Push, SW9 SW_Push, U1 ATmega644P-20P, U2 74HC238, X2 CXO_DIP8

Commit message: Keyboard code and schematics
Updated the Schematics and have a mostly functioning keyboard (can't turn off caps lock yet)
Parts:
- DS1: value HDSP-2503 -> HDSP-2103
- SW1, SW10, SW11, SW12, SW13, SW14, SW15, SW16, SW17, SW18, SW19, SW2, SW20, SW21, SW22, SW23, SW24, SW25, SW26, SW27, SW28, SW29, SW3, SW30, SW31, SW32, SW33, SW34, SW35, SW36, SW37, SW38, SW39, SW4, SW40, SW41, SW42, SW43, SW44, SW45, SW46, SW47, SW49, SW5, SW50, SW51, SW52, SW54, SW56, SW58, SW59, SW6, SW60, SW61, SW62, SW63, SW64, SW7, SW8, SW9: footprint Button_Switch_Keyboard:SW_Cherry_MX_1.00u_PCB -> PaulasKiCADFootPrint:SW_Cherry_MX_1.00u_PCB_LED
- SW48: footprint Button_Switch_Keyboard:SW_Cherry_MX_6.25u_PCB -> PaulasKiCADFootPrint:SW_Cherry_MX_1.00u_PCB_LED
- SW53, SW65: footprint Button_Switch_Keyboard:SW_Cherry_MX_2.00u_PCB -> PaulasKiCADFootPrint:SW_Cherry_MX_1.00u_PCB_LED
- SW55: footprint Button_Switch_Keyboard:SW_Cherry_MX_ISOEnter_PCB -> PaulasKiCADFootPrint:SW_Cherry_MX_1.00u_PCB_LED
- SW57: footprint Button_Switch_Keyboard:SW_Cherry_MX_1.50u_PCB -> PaulasKiCADFootPrint:SW_Cherry_MX_1.00u_PCB_LED
- U2: value 74HC238 -> 74HC138
