File: Schematics/PC6502-KEYTFT/PC6502-KEYTFT.kicad_sch (KiCad schematic)
At the start: 66 parts, among them J1 BUS, J2 Conn_02x20_Odd_Even, J3 Conn_01x03, J4 Conn_02x05_Odd_Even, J5 Conn_02x05_Odd_Even, J6 MTJ-88ARX1-FSM-LG, Q1 BSS138, Q2 BSS138, Q3 BSS138, Q4 BSS138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

Commit message: KeyTFT to Rev 1.1
COmplete revamp of Schamtic and PCB, to make things simpler, and hopefully a bit quicker.
Parts:
- removed J3: Conn_01x03, Connector_PinHeader_2.54mm:PinHeader_1x03_P2.54mm_Vertical, symbol Connector_Generic:Conn_01x03
- removed J4: Conn_02x05_Odd_Even, Connector_PinHeader_2.54mm:PinHeader_2x05_P2.54mm_Vertical, symbol Connector_Generic:Conn_02x05_Odd_Even
- removed Q1, Q2, Q3, Q4, Q5, Q6: BSS138, Package_TO_SOT_SMD:SOT-23, symbol Transistor_FET:BSS138
- removed R10, R12, R14, R15, R16, R18, R20, R21, R22, R23, R24, R25, R26, R46, R5, R8: 4.7K, Resistor_SMD:R_0603_1608Metric, symbol Device:R
- removed R13, R17, R19, R4, R6, R9: 1.8K, Resistor_SMD:R_0603_1608Metric, symbol Device:R
- removed R7: 3K3, Resistor_SMD:R_0603_1608Metric_Pad0.98x0.95mm_HandSolder, symbol Device:R
- removed U1: ATmega644P-20P, Package_DIP:DIP-40_W15.24mm, symbol MCU_Microchip_ATmega:ATmega644P-20P
- added C48, C49, C5: 100nF, Capacitor_SMD:C_0603_1608Metric, symbol Device:C
- added C9: 10uF, Capacitor_SMD:C_0805_2012Metric, symbol Device:C
- added D17: 1N4148, Diode_THT:D_DO-35_SOD27_P7.62mm_Horizontal, symbol Diode:1N4148
- added R67, R68: 0R, Resistor_SMD:R_0603_1608Metric, symbol Device:R
- added R82: 3K3, Resistor_SMD:R_0603_1608Metric, symbol Device:R
- added TP1, TP2: TestPoint, TestPoint:TestPoint_Loop_D1.80mm_Drill1.0mm_Beaded, symbol Connector:TestPoint
- added U1: W65C51NxP, Package_DIP:DIP-28_W15.24mm, symbol 65xx-library:W65C51NxP
- added U8, U9: TXB0108PW, Package_SO:TSSOP-20_4.4x6.5mm_P0.65mm, symbol Logic_LevelTranslator:TXB0108PW
- C2, C3, C4, C8: footprint Capacitor_SMD:C_0805_2012Metric -> Capacitor_SMD:C_0603_1608Metric
- C7: value 0.1u -> 100nF; LCSC (none) -> C49678; Manufacturer Kemet -> (none); ManufacturerPN C0603C104K3RAC7867 -> (none)
- R1, R11, R29, R30: footprint Resistor_SMD:R_0603_1608Metric_Pad0.98x0.95mm_HandSolder -> Resistor_SMD:R_0603_1608Metric
- R2, R3: value 4.7K -> 0R; footprint Resistor_SMD:R_0603_1608Metric -> Resistor_SMD:R_0603_1608Metric_Pad0.98x0.95mm_HandSolder; LCSC DNF -> C23179
- R27, R28: value 10K -> 3K3; footprint Resistor_SMD:R_0603_1608Metric_Pad0.98x0.95mm_HandSolder -> Resistor_SMD:R_0603_1608Metric
- X2: value CXO_DIP8 -> 1.8432MHz
Connections:
- net +3.3V: now also C7.1, C5.1, U8.10 (OE), U8.2 (V_{CCA}), U9.10 (OE), U9.2 (V_{CCA}); no longer R2.1
- net +5V: now also C48.1, C49.1, C9.1, R82.1, U1.15 (VCC), U1.2 (CS1), U8.19 (V_{CCB}), U9.19 (V_{CCB}); no longer C7.1, R3.1
- net A0: now also U1.13 (RS0), U8.13 (B7)
- net A1: now also U2.6 (I/O), U1.14 (RS1)
- net D0: now also U2.41 (I/O/GCLK3), U1.18 (D0), U9.20 (B1); no longer U2.36 (I/O)
- net D1: now also U2.36 (I/O), U1.19 (D1), U9.18 (B2); no longer U2.34 (I/O)
- net D2: now also U2.34 (I/O), U1.20 (D2), U9.17 (B3)
- net D3: now also U1.21 (D3), U9.16 (B4)
- net D4: now also U1.22 (D4), U9.15 (B5)
- net D5: now also U1.23 (D5), U9.14 (B6)
- net D6: now also U1.24 (D6), U9.13 (B7)
- net D7: now also U1.25 (D7), U9.12 (B8)
- net GND: now also C48.2, C49.2, C5.2, C9.2, TP1.1, U1.1 (VSS), U1.16 (~{DCD}), U1.17 (~{DSR}), U1.9 (~{CTS}), U8.11 (GND), U9.11 (GND)
- net KEY_nCS: now also U1.3 (~{CS2})
- net RnW: now also U1.28 (R/~{W}), U8.15 (B5)
- net SYSCLK: now also U1.27 (ϕ2)
- net nIRQ: now also D17.2 (A)
- net nRES: now also U1.4 (~{RES})
- net at X2.5 (OUT): now also U1.6 (XTAL1)
- net at U2.33 (I/O): now also TP2.1
- net DISP_nRES: now reaches U2.37 (I/O)
- net DISP_nRES: now also U8.16 (B4)
- net DISP_EN: now reaches U2.39 (I/O)
- net DISP_EN: now also U8.20 (B1)
- net BL: now reaches U2.40 (I/O)
- net BL: now also U8.12 (B8)
- net 3V3_D0: now reaches J2.15 (Pin_15)
- net 3V3_D0: now also U9.1 (A1)
- net 3V3_D1: now reaches J2.16 (Pin_16)
- net 3V3_D1: now also U9.3 (A2)
- net 3V3_D2: now reaches J2.17 (Pin_17)
- net 3V3_D2: now also U9.4 (A3)
- net 3V3_D3: now reaches J2.18 (Pin_18)
- net 3V3_D3: now also U9.5 (A4)
- net 3V3_D4: now reaches J2.19 (Pin_19)
- net 3V3_D4: now also U9.6 (A5)
- net 3V3_D5: now reaches J2.20 (Pin_20)
- net 3V3_D5: now also U9.7 (A6)
- net 3V3_D6: now reaches J2.21 (Pin_21)
- net 3V3_D6: now also U9.8 (A7)
- net 3V3_D7: now reaches J2.22 (Pin_22)
- net 3V3_D7: now also U9.9 (A8)
- net at X2.1 (EN): now also R82.2
- net 3V3_CP_nINT: no longer names the net of J2.33 (Pin_33)
- net 3V3_CP_nRST: no longer names the net of J2.36 (Pin_36)
- net 3V3_SCL: no longer names the net of J2.35 (Pin_35)
- net 3V3_SCL: no longer R2.2
- net 3V3_SDA: no longer names the net of J2.34 (Pin_34)
- net 3V3_SPI_CLK renamed 3V3_RS
- net 3V3_RS: now also U8.8 (A7)
- net 3V3_SPI_MISO renamed 3V3_RnW
- net 3V3_RnW: now also U8.6 (A5)
- net 3V3_SPI_MOSI renamed 3V3_nCS
- net 3V3_nCS: now also U8.3 (A2)
- net 3V3_SPI_nCS renamed 3V3_EN
- net 3V3_EN: now also U8.1 (A1)
- net 3V3_TFT_BL: no longer names the net of J2.14 (Pin_14)
- net 3V3_TFT_BL: now also R68.2
- net 3V3_TFT_INT renamed 3V3_nINT
- net 3V3_nINT: now also U8.7 (A6)
- net 3V3_TFT_nBUSY renamed 3V3_nWAIT
- net 3V3_nWAIT: now also U8.4 (A3)
- net 3V3_TFT_nRST renamed 3V3_nRES
- net 3V3_nRES: now also R67.2
- net 5V_SCL renamed SER_RX
- net SER_RX: now also R28.2, U1.12 (RxD)
- net KEY_SER_IN: no longer names the net of J6.3
- net KEY_SER_IN: now also R3.1; no longer R27.2
- net KEY_SER_OUT: no longer names the net of J6.5
- net KEY_SER_OUT: now also R2.1; no longer R28.2
- net TFT_nCS renamed DISP_nCS
- net DISP_nCS: now also U8.18 (B2)
- net nRXF renamed DISP_nWAIT
- net DISP_nWAIT: now also U8.17 (B3)
- net nTXE renamed DISP_nINT
- net DISP_nINT: now also U8.14 (B6)
- new net: R67.1, U8.5 (A4)
- new net: D17.1 (K), U1.26 (~{IRQ})
- new net 3V3_BL: R68.1, U8.9 (A8)
- new net SER_TX: R2.2, R27.2, U1.10 (TxD)
- no-connect marks 27 -> 25
Other:
- note added: "Arrange close so that resistors can be rotated 90 degrees to swap RX and TX lines, just in case."
- note added: "With 6800 interface and 5V Supply."
- note removed: "20Mhz"
- moved on the sheet: C1, C11, C2, C3, C4, C6, C8, D3, D4, H3, H4, H5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
