File: Schematics/PC6502-KEYTFT/PC6502-KEYTFT.kicad_pcb (KiCad board)
At the start: 4 copper layers, 100 x 100 mm, 66 parts, among them J1 BUS, J2 Conn_02x20_Odd_Even, J3 Conn_01x03, J4 Conn_02x05_Odd_Even, J5 Conn_02x05_Odd_Even, J6 MTJ-88ARX1-FSM-LG, Q1 BSS138, Q2 BSS138, Q3 BSS138, Q4 BSS138, Q5 BSS138, Q6 BSS138, Q7 2N3904, Q8 2N3904, U1 ATmega644P-20P, U2 ATF1502AS, U21 AMS1117-3.3, X2 CXO_DIP8

Commit message: KeyTFT to Rev 1.1
COmplete revamp of Schamtic and PCB, to make things simpler, and hopefully a bit quicker.
Parts:
- removed J3: Conn_01x03, Connector_PinHeader_2.54mm:PinHeader_1x03_P2.54mm_Vertical
- removed J4: Conn_02x05_Odd_Even, Connector_PinHeader_2.54mm:PinHeader_2x05_P2.54mm_Vertical
- removed Q1, Q2, Q3, Q4, Q5, Q6: BSS138, Package_TO_SOT_SMD:SOT-23
- removed R10, R12, R14, R15, R16, R18, R20, R21, R22, R23, R24, R25, R26, R46, R5, R8: 4.7K, Resistor_SMD:R_0603_1608Metric
- removed R13, R17, R19, R4, R6, R9: 1.8K, Resistor_SMD:R_0603_1608Metric
- removed R7: 3K3, Resistor_SMD:R_0603_1608Metric_Pad0.98x0.95mm_HandSolder
- added C48: 100nF, Capacitor_SMD:C_0603_1608Metric, F.Cu at (131.2, 82.1)
- added C49: 100nF, Capacitor_SMD:C_0603_1608Metric, F.Cu at (181.7, 65.5)
- added C5: 100nF, Capacitor_SMD:C_0603_1608Metric, F.Cu at (172.8, 100.5)
- added C9: 10uF, Capacitor_SMD:C_0805_2012Metric, F.Cu at (183.7, 65.4)
- added D17: 1N4148, Diode_THT:D_DO-35_SOD27_P7.62mm_Horizontal, F.Cu at (116.1, 87.0)
- added R67: 0R, Resistor_SMD:R_0603_1608Metric, F.Cu at (178.1, 99.7)
- added R68: 0R, Resistor_SMD:R_0603_1608Metric, F.Cu at (178.1, 96.5)
- added R82: 3K3, Resistor_SMD:R_0603_1608Metric, F.Cu at (147.0, 66.8)
- added TP1: TestPoint, TestPoint:TestPoint_Loop_D1.80mm_Drill1.0mm_Beaded, F.Cu at (192.1, 57.4)
- added TP2: TestPoint, TestPoint:TestPoint_Loop_D1.80mm_Drill1.0mm_Beaded, F.Cu at (135.1, 141.7)
- added U8: TXB0108PW, Package_SO:TSSOP-20_4.4x6.5mm_P0.65mm, F.Cu at (168.0, 103.6)
- added U9: TXB0108PW, Package_SO:TSSOP-20_4.4x6.5mm_P0.65mm, F.Cu at (168.0, 91.2)
- C2, C3, C4, C8: footprint Capacitor_SMD:C_0805_2012Metric -> Capacitor_SMD:C_0603_1608Metric
- C7: value 0.1u -> 100nF
- R1, R11, R29, R30: footprint Resistor_SMD:R_0603_1608Metric_Pad0.98x0.95mm_HandSolder -> Resistor_SMD:R_0603_1608Metric
- R2, R3: value 4.7K -> 0R; footprint Resistor_SMD:R_0603_1608Metric -> Resistor_SMD:R_0603_1608Metric_Pad0.98x0.95mm_HandSolder
- R27, R28: value 10K -> 3K3; footprint Resistor_SMD:R_0603_1608Metric_Pad0.98x0.95mm_HandSolder -> Resistor_SMD:R_0603_1608Metric
- U1: value ATmega644P-20P -> W65C51NxP; footprint Package_DIP:DIP-40_W15.24mm -> Package_DIP:DIP-28_W15.24mm
- X2: value CXO_DIP8 -> 1.8432MHz
- moved R3 52.1 mm to (141.4, 52.8), turned to 180 degrees
- moved R2 48.0 mm to (141.4, 54.6), turned to 0 degrees
- moved C3 42.9 mm to (172.8, 106.6)
- moved C4 37.6 mm to (172.9, 94.4)
- moved C7 32.5 mm to (172.8, 88.9), turned to -90 degrees
- moved X2 31.7 mm to (142.8, 63.3), turned to 180 degrees
- moved U1 27.4 mm to (128.8, 83.5), turned to 180 degrees
- moved C1 26.0 mm to (167.3, 81.7)
- moved C11 26.0 mm to (171.7, 81.6)
- moved U21 26.0 mm to (169.6, 76.2)
- moved R30 9.72 mm to (158.9, 64.2), turned to -90 degrees
- moved R27 7.15 mm to (151.8, 64.2)
- moved R29 4.64 mm to (171.4, 64.0), turned to -90 degrees
- moved C2 2.04 mm to (138.8, 140.9)
- moved J5 2.03 mm to (160.2, 128.3)
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Connections:
- C7 pad 1: +5V -> +3.3V
- D2 pad 1: TFT_nCS -> DISP_nCS
- J2 pad 10: 3V3_TFT_INT -> 3V3_nINT
- J2 pad 11: 3V3_TFT_nRST -> /3V3_nRES
- J2 pad 14: 3V3_TFT_BL -> Net-(J2-Pin_14)
- J2 pad 15: unconnected-(J2-Pin_15-Pad15) -> /3V3_D0
- J2 pad 16: unconnected-(J2-Pin_16-Pad16) -> /3V3_D1
- J2 pad 17: unconnected-(J2-Pin_17-Pad17) -> /3V3_D2
- J2 pad 18: unconnected-(J2-Pin_18-Pad18) -> /3V3_D3
- J2 pad 19: unconnected-(J2-Pin_19-Pad19) -> /3V3_D4
- J2 pad 20: unconnected-(J2-Pin_20-Pad20) -> /3V3_D5
- J2 pad 21: unconnected-(J2-Pin_21-Pad21) -> /3V3_D6
- J2 pad 22: unconnected-(J2-Pin_22-Pad22) -> /3V3_D7
- J2 pad 33: 3V3_CP_nINT -> unconnected-(J2-Pin_33-Pad33)
- J2 pad 34: 3V3_SDA -> unconnected-(J2-Pin_34-Pad34)
- J2 pad 35: 3V3_SCL -> unconnected-(J2-Pin_35-Pad35)
- J2 pad 36: 3V3_CP_nRST -> unconnected-(J2-Pin_36-Pad36)
- J2 pad 5: 3V3_SPI_nCS -> /3V3_EN
- J2 pad 6: 3V3_SPI_MISO -> 3V3_RnW
- J2 pad 7: 3V3_SPI_MOSI -> /3V3_nCS
- J2 pad 8: 3V3_SPI_CLK -> 3V3_RS
- J2 pad 9: 3V3_TFT_nBUSY -> /3V3_nWAIT
- J6 pad 3: KEY_SER_IN -> Net-(J6-Pad3)
- J6 pad 5: KEY_SER_OUT -> Net-(J6-Pad5)
- R2 pad 1: +3.3V -> Net-(J6-Pad5)
- R2 pad 2: 3V3_SCL -> SER_TX
- R27 pad 2: KEY_SER_IN -> SER_TX
- R28 pad 2: KEY_SER_OUT -> SER_RX
- R3 pad 1: +5V -> Net-(J6-Pad3)
- R3 pad 2: 5V_SCL -> SER_RX
- U1 pad 1: Net-(Q4-D) -> GND
- U1 pad 10: +5V -> SER_TX
- U1 pad 11: GND -> unconnected-(U1-~{DTR}-Pad11)
- U1 pad 12: unconnected-(U1-XTAL2-Pad12) -> SER_RX
- U1 pad 13: Net-(U1-XTAL1) -> /A0
- U1 pad 14: KEY_SER_IN -> /A1
- U1 pad 15: KEY_SER_OUT -> +5V
- U1 pad 16: /A1 -> GND
- U1 pad 17: /A0 -> GND
- U1 pad 18: nRXF -> /D0
- U1 pad 19: nTXE -> /D1
- U1 pad 2: 5V_TFT_nBUSY -> +5V
- U1 pad 20: KEY_nCS -> /D2
- U1 pad 21: TFT_nCS -> /D3
- U1 pad 22: 5V_SCL -> /D4
- U1 pad 23: 5V_SDA -> /D5
- U1 pad 24: AVR_TCK -> /D6
- U1 pad 25: AVR_TMS -> /D7
- U1 pad 26: AVR_TDO -> Net-(D17-K)
- U1 pad 27: AVR_TDI -> SYSCLK
- U1 pad 28: 5V_CP_nINT -> RnW
- U1 pad 3: RnW -> KEY_nCS
- U1 pad 4: 5V_TFT_BL -> nRES
- U1 pad 5: SPI_nCS -> unconnected-(U1-RxC-Pad5)
- U1 pad 6: SPI_MOSI -> Net-(U1-XTAL1)
- U1 pad 7: SPI_MISO -> unconnected-(U1-XTAL2-Pad7)
- U1 pad 8: SPI_CLK -> unconnected-(U1-~{RTS}-Pad8)
- U1 pad 9: AVR_nRST -> GND
- U2 pad 1: nRXF -> DISP_nWAIT
- U2 pad 29: TFT_nCS -> DISP_nCS
- U2 pad 33: unconnected-(U2-I/O-Pad33) -> Net-(TP2-Pad1)
- U2 pad 34: /D1 -> /D2
- U2 pad 36: /D0 -> /D1
- U2 pad 37: unconnected-(U2-I/O-Pad37) -> DISP_nRES
- U2 pad 39: unconnected-(U2-I/O-Pad39) -> DISP_EN
- U2 pad 40: unconnected-(U2-I/O-Pad40) -> BL
- U2 pad 41: unconnected-(U2-I/O/GCLK3-Pad41) -> /D0
- U2 pad 44: nTXE -> DISP_nINT
- U2 pad 6: unconnected-(U2-I/O-Pad6) -> /A1
Routing:
- net DISP_nCS: track 0.00 -> 126.3 mm, vias 0 -> 4
- net /D2: track 35.0 -> 135.9 mm, vias 0 -> 3
- net TFT_nCS: track 99.0 -> 0.00 mm, vias 2 -> 0
- net SPI_nCS: track 97.4 -> 0.00 mm, vias 6 -> 0
- net SPI_MOSI: track 97.0 -> 0.00 mm, vias 6 -> 0
- net SPI_CLK: track 96.9 -> 0.00 mm, vias 6 -> 0
- net SPI_MISO: track 96.8 -> 0.00 mm, vias 6 -> 0
- net Net-(Q4-D): track 94.6 -> 0.00 mm, vias 4 -> 0
- net 5V_TFT_nBUSY: track 93.2 -> 0.00 mm, vias 4 -> 0
- net 5V_TFT_BL: track 86.1 -> 0.00 mm, vias 6 -> 0
- net /A1: track 33.1 -> 116.8 mm, vias 2 -> 3
- net KEY_SER_OUT: track 81.4 -> 0.00 mm, vias 3 -> 0
- net KEY_SER_IN: track 78.7 -> 0.00 mm, vias 3 -> 0
- net 5V_CP_nRST: track 78.3 -> 0.00 mm, vias 3 -> 0
- net 3V3_SDA: track 68.6 -> 0.00 mm, vias 2 -> 0
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Other:
- board text added: "GND"
- board text added: "U1"
- board text added: "V1.1 Nov 2025"
- board text removed: "AVR-JTAG"
- board text removed: "V1.0 Oct 2025"

Commit message: Updated KeyTFT Schematic to include mods
Parts:
- added R4: 3K3, Resistor_SMD:R_0603_1608Metric, F.Cu at (157.5, 87.6)
- added R5: 1K8, Resistor_SMD:R_0603_1608Metric, F.Cu at (161.7, 87.6)
- U8, U9: value TXB0108PW -> TXS0108EPW
Connections:
- net Net-(TP2-Pad1) renamed /TXS_OE_5V
- J2 pad 23: unconnected-(J2-Pin_23-Pad23) -> GND
- J2 pad 24: unconnected-(J2-Pin_24-Pad24) -> GND
- J2 pad 25: unconnected-(J2-Pin_25-Pad25) -> GND
- J2 pad 26: unconnected-(J2-Pin_26-Pad26) -> GND
- J2 pad 27: unconnected-(J2-Pin_27-Pad27) -> GND
- J2 pad 28: unconnected-(J2-Pin_28-Pad28) -> GND
- J2 pad 29: unconnected-(J2-Pin_29-Pad29) -> GND
- J2 pad 30: unconnected-(J2-Pin_30-Pad30) -> GND
- U9 pad 10: +3.3V -> TXS_OE
Routing:
- net /TXS_OE_5V: track 6.01 -> 83.3 mm, vias 0 -> 2
- net +3.3V: track 69.4 -> 57.5 mm, vias 6 -> 5
- net TXS_OE: track 0.00 -> 7.57 mm
- net +5V: track 52.2 -> 49.9 mm
- net GND: vias 24 -> 37
Other:
- board text added: "V1.2 Dec 2025"
- board text removed: "V1.1 Nov 2025"

Commit message: Changes I forgot to commit
Parts:
- R4: value 3K3 -> 1K8
- R5: value 1K8 -> 3K3
Changed lines of the file:
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@@
 			)
 		)
-		(property "Value" "3K3"
+		(property "Value" "1K8"
 			(at 0 1.43 90)
 			(layer "F.Fab")
@@
 			)
 		)
-		(property "Value" "1K8"
+		(property "Value" "3K3"
 			(at 0 1.43 90)
 			(layer "F.Fab")
